File: nnv2-toupee/nnv2-toupee.kicad_pcb (KiCad board)
At the start: 2 copper layers, 71.5 x 29.4 mm, 5 parts, among them J1 Conn_01x02_Socket, J2 Conn_01x04_Socket, J3 Conn_01x04_Pin, SW1 SW_SPST, U1 Nice! Nano (ProMicro)

Commit message: working towards a comb over
Parts:
- moved J1 20.4 mm to (204.3, 72.3)
- moved J2 14.8 mm to (176.9, 72.3), turned to 0 degrees
- moved U1 3.57 mm to (208.6, 78.8)
- moved SW1 2.60 mm to (210.3, 86.5)
Routing:
- net VCC: track 52.6 -> 102.2 mm
- net /SCL: track 47.8 -> 70.3 mm
- net /SDA: track 71.4 -> 61.4 mm
- net /rawswitch: track 13.1 -> 17.7 mm
Other:
- board size 71.5 x 29.4 mm -> 71.5 x 35.7 mm
